File: pcb/controls-board/controls.sch (KiCad schematic (older format))
At the start: 4 parts, among them J1 CONTROLS_HEADER, J2 ENCODER, SW1 PARAM BUTTON, SW2 MODE BUTTON

Commit message: working on finding components for parts
Parts:
- removed J1: CONTROLS_HEADER, symbol CONTROLS_HEADER
- added D?: LED_RABG, symbol LED_RABG
- added J?: CONTROLS_HEADER, symbol CONTROLS_HEADER
Connections:
- net at J2.2 (ENC_CW): now also J?.2 (ENC_CW)
- net at J2.3 (ENC_CCW): now also J?.3 (ENC_CCW)
- net at SW2.2: now also J2.1 (GND), SW1.2, J?.1 (GND)
- new net: J?.4 (MODE), SW2.1
- new net: J?.5 (PARAM), SW1.1
- new net: D?.1 (RED_CATHODE), J?.6 (LED_R)
- new net: D?.4 (GREEN_CATHODE), J?.7 (LED_G)
- new net: D?.3 (BLUE_CATHODE), J?.8 (LED_B)
- new net: D?.2 (COMMON_ANODE), J?.9 (LED_5V)
Other:
- moved on the sheet: SW1, SW2
Changed lines of the file:
@@
 EESchema Schematic File Version 2
+LIBS:controls-components
 LIBS:power
 LIBS:device
@@
 LIBS:memory
 LIBS:xilinx
-LIBS:special
 LIBS:microcontrollers
 LIBS:dsp
@@
 LIBS:contrib
 LIBS:valves
-LIBS:controls-components
 LIBS:controls-cache
-EELAYER 27 0
+EELAYER 25 0
 EELAYER END
 $Descr A4 11693 8268
@@
 $EndDescr
 $Comp
-L CONTROLS_HEADER J1
-U 1 1 5529C30F
-P 4700 3850
-F 0 "J1" H 4700 3400 60  0000 C CNN
-F 1 "CONTROLS_HEADER" H 4700 4500 60  0000 C CNN
-F 2 "" H 4650 3850 60  0000 C CNN
-F 3 "" H 4650 3850 60  0000 C CNN
-	1    4700 3850
-	-1   0    0    -1
-$EndComp
-$Comp
 L ENCODER J2
 U 1 1 5529C488
@@
 L SW_PUSH SW2
 U 1 1 5529C4A4
-P 6100 4150
-F 0 "SW2" H 6250 4260 50  0000 C CNN
-F 1 "MODE BUTTON" H 6100 4070 50  0000 C CNN
-F 2 "~" H 6100 4150 60  0000 C CNN
-F 3 "~" H 6100 4150 60  0000 C CNN
-	1    6100 4150
+P 5950 3000
+F 0 "SW2" H 6100 3110 50  0000 C CNN
+F 1 "MODE BUTTON" H 5950 2920 50  0000 C CNN
+F 2 "~" H 5950 3000 60  0000 C CNN
+F 3 "~" H 5950 3000 60  0000 C CNN
+	1    5950 3000
 	0    -1   -1   0
+$EndComp
+Wire Wire Line
+	6100 3400 5200 3400
+Connection ~ 5350 3400
+Wire Wire Line
+	5200 3700 6100 3700
+Wire Wire Line
+	6100 3550 5200 3550
+$Comp
+L CONTROLS_HEADER J?
+U 1 1 58046964
+P 4700 3850
+F 0 "J?" H 4700 2750 60  0000 C CNN
+F 1 "CONTROLS_HEADER" H 4700 4500 60  0000 C CNN
+F 2 "" H 4500 3850 60  0000 C CNN
+F 3 "" H 4500 3850 60  0000 C CNN
+	1    4700 3850
+	-1   0    0    -1
 $EndComp
 $Comp
 L SW_PUSH SW1
 U 1 1 5529C4B3
-P 5700 4300
-F 0 "SW1" H 5850 4410 50  0000 C CNN
-F 1 "PARAM BUTTON" H 5700 4220 50  0000 C CNN
-F 2 "~" H 5700 4300 60  0000 C CNN
-F 3 "~" H 5700 4300 60  0000 C CNN
-	1    5700 4300
+P 5600 3000
+F 0 "SW1" H 5750 3110 50  0000 C CNN
+F 1 "PARAM BUTTON" H 5600 2920 50  0000 C CNN
+F 2 "~" H 5600 3000 60  0000 C CNN
+F 3 "~" H 5600 3000 60  0000 C CNN
+	1    5600 3000
 	0    -1   -1   0
 $EndComp
 Wire Wire Line
-	6100 3400 5200 3400
+	5350 3400 5350 2700
 Wire Wire Line
-	5350 3400 5350 4600
+	5350 2700 5950 2700
+Connection ~ 5600 2700
 Wire Wire Line
-	5350 4600 6100 4600
-Connection ~ 5350 3400
+	5200 3850 5950 3850
 Wire Wire Line
-	6100 4600 6100 4450
-Connection ~ 5700 4600
+	5950 3850 5950 3300
 Wire Wire Line
-	5700 4000 5200 4000
+	5200 4000 5600 4000
 Wire Wire Line
-	6100 3850 5200 3850
+	5600 4000 5600 3300
 Wire Wire Line
-	5200 3700 6100 3700
+	5200 4150 5800 4150
 Wire Wire Line
-	6100 3550 5200 3550
+	5200 4300 5650 4300
+Wire Wire Line
+	5200 4450 5500 4450
+Wire Wire Line
+	5200 4600 5300 4600
+Wire Wire Line
+	5300 4600 5300 4900
+Wire Wire Line
+	5300 4900 6400 4900
+Wire Wire Line
+	6400 4900 6400 4350
+Wire Wire Line
+	5650 4300 5650 4350
+Wire Wire Line
+	5650 4350 5800 4350
+Wire Wire Line
+	5500 4450 5500 4550
+Wire Wire Line
+	5500 4550 5800 4550
+$Comp
+L LED_RABG D?
+U 1 1 580C0207
+P 6100 4350
+F 0 "D?" H 6175 4700 50  0000 C CNN
+F 1 "LED_RABG" H 6125 4000 50  0000 C CNN
+F 2 "" H 6050 4300 50  0000 C CNN
+F 3 "" H 6050 4300 50  0000 C CNN
+	1    6100 4350
+	1    0    0    -1
+$EndComp
 $EndSCHEMATC

Commit message: finished choosing components for main board
Parts:
- D?: Manufacturer (none) -> Adafruit Industries LLC; Order (none) -> No; Product code (none) -> 314; Product description (none) -> Red, Green, Blue (RGB) LED Indication - Discrete 2.1V Red, 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; Supplier (none) -> Digikey; Supplier URL (none) -> http://www.digikey.co.uk/product-detail/en/adafruit-industr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; Supplier code (none) -> 1528-1127-ND
Changed lines of the file:
@@
 F 2 "" H 6050 4300 50  0000 C CNN
 F 3 "" H 6050 4300 50  0000 C CNN
+F 4 "Adafruit Industries LLC" H 6100 4350 60  0001 C CNN "Manufacturer"
+F 5 "Red, Green, Blue (RGB) LED Indication - Discrete 2.1V Red, 3.8V Green, 2.7V Blue 4-DIP (0.200\", 5.08mm)" H 6100 4350 60  0001 C CNN "Product description"
+F 6 "314" H 6100 4350 60  0001 C CNN "Product code"
+F 7 "Digikey" H 6100 4350 60  0001 C CNN "Supplier"
+F 8 "1528-1127-ND" H 6100 4350 60  0001 C CNN "Supplier code"
+F 9 "No" H 6100 4350 60  0001 C CNN "Order"
+F 10 "http://www.digikey.co.uk/product-detail/en/adafruit-industries-llc/314/1528-1127-ND/5353587" H 6100 4350 60  0001 C CNN "Supplier URL"
 	1    6100 4350
 	1    0    0    -1

Commit message: found components for controls board
Parts:
- removed SW1: PARAM BUTTON, ~, symbol SW_PUSH
- added SW?: PARAM BUTTON, ~, symbol SW_PUSH
- J2: Manufacturer (none) -> TT Electronics/BI; Order (none) -> No; Product code (none) -> EN12-HN22AF25; Product description (none) -> ENCODER 12MM ROTARY TOP ADJUST; Supplier (none) -> Digikey; Supplier URL (none) -> http://www.digikey.co.uk/product-detail/en/tt-electronics-b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; Supplier code (none) -> 987-1399-ND
- J?: Manufacturer (none) -> On Shore Technology Inc.; Order (none) -> No; Product code (none) -> 302-S101; Product description (none) -> 10 Positions Header, Shrouded Connector 0.100\" (2.54mm) Th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; Supplier (none) -> Digikey; Supplier URL (none) -> http://www.digikey.co.uk/product-detail/en/on-shore-technol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; Supplier code (none) -> ED1543-ND
- SW2: Manufacturer (none) -> C&K Components; Order (none) -> No; Product code (none) -> D6R40 F1 LFS; Product description (none) -> Pushbutton SwPushbutton Switch SPST-NO Keyswitch Through Ho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; Supplier (none) -> Digikey; Supplier URL (none) -> http://www.digikey.co.uk/product-detail/en/c-k-components/D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; Supplier code (none) -> 401-1975-ND
Connections:
- net at J2.1 (GND), J?.1 (GND), SW2.2: now also SW?.2
- net at J?.5 (PARAM): now also SW?.1
Changed lines of the file:
@@
 F 2 "" H 6450 3450 60  0000 C CNN
 F 3 "" H 6450 3450 60  0000 C CNN
+F 4 "TT Electronics/BI" H 6650 3550 60  0001 C CNN "Manufacturer"
+F 5 "ENCODER 12MM ROTARY TOP ADJUST" H 6650 3550 60  0001 C CNN "Product description"
+F 6 "EN12-HN22AF25" H 6650 3550 60  0001 C CNN "Product code"
+F 7 "Digikey" H 6650 3550 60  0001 C CNN "Supplier"
+F 8 "987-1399-ND" H 6650 3550 60  0001 C CNN "Supplier code"
+F 9 "No" H 6650 3550 60  0001 C CNN "Order"
+F 10 "http://www.digikey.co.uk/product-detail/en/tt-electronics-bi/EN12-HN22AF25/987-1399-ND/2620668" H 6650 3550 60  0001 C CNN "Supplier URL"
 	1    6650 3550
 	1    0    0    -1
-$EndComp
-$Comp
-L SW_PUSH SW2
-U 1 1 5529C4A4
-P 5950 3000
-F 0 "SW2" H 6100 3110 50  0000 C CNN
-F 1 "MODE BUTTON" H 5950 2920 50  0000 C CNN
-F 2 "~" H 5950 3000 60  0000 C CNN
-F 3 "~" H 5950 3000 60  0000 C CNN
-	1    5950 3000
-	0    -1   -1   0
 $EndComp
 Wire Wire Line
@@
 F 2 "" H 4500 3850 60  0000 C CNN
 F 3 "" H 4500 3850 60  0000 C CNN
+F 4 "On Shore Technology Inc." H 4700 3850 60  0001 C CNN "Manufacturer"
+F 5 "10 Positions Header, Shrouded Connector 0.100\" (2.54mm) Through Hole Gold" H 4700 3850 60  0001 C CNN "Product description"
+F 6 "302-S101" H 4700 3850 60  0001 C CNN "Product code"
+F 7 "Digikey" H 4700 3850 60  0001 C CNN "Supplier"
+F 8 "ED1543-ND" H 4700 3850 60  0001 C CNN "Supplier code"
+F 9 "No" H 4700 3850 60  0001 C CNN "Order"
+F 10 "http://www.digikey.co.uk/product-detail/en/on-shore-technology-inc/302-S101/ED1543-ND/2178422" H 4700 3850 60  0001 C CNN "Supplier URL"
 	1    4700 3850
 	-1   0    0    -1
-$EndComp
-$Comp
-L SW_PUSH SW1
-U 1 1 5529C4B3
-P 5600 3000
-F 0 "SW1" H 5750 3110 50  0000 C CNN
-F 1 "PARAM BUTTON" H 5600 2920 50  0000 C CNN
-F 2 "~" H 5600 3000 60  0000 C CNN
-F 3 "~" H 5600 3000 60  0000 C CNN
-	1    5600 3000
-	0    -1   -1   0
 $EndComp
 Wire Wire Line
@@
 	1    0    0    -1
 $EndComp
+$Comp
+L SW_PUSH SW?
+U 1 1 580D518A
+P 5600 3000
+F 0 "SW?" H 5750 3110 50  0000 C CNN
+F 1 "PARAM BUTTON" H 5600 2920 50  0000 C CNN
+F 2 "~" H 5600 3000 60  0000 C CNN
+F 3 "~" H 5600 3000 60  0000 C CNN
+F 4 "C&K Components" H 5600 3000 60  0001 C CNN "Manufacturer"
+F 5 "Pushbutton Switch SPST-NO Keyswitch Through Hole" H 5600 3000 60  0001 C CNN "Product description"
+F 6 "D6R50 F1 LFS" H 5600 3000 60  0001 C CNN "Product code"
+F 7 "Digikey" H 5600 3000 60  0001 C CNN "Supplier"
+F 8 "401-1976-ND" H 5600 3000 60  0001 C CNN "Supplier code"
+F 9 "No" H 5600 3000 60  0001 C CNN "Order"
+F 10 "http://www.digikey.co.uk/product-detail/en/c-k-components/D6R50-F1-LFS/401-1976-ND/1466333" H 5600 3000 60  0001 C CNN "Supplier URL"
+	1    5600 3000
+	0    -1   -1   0
+$EndComp
+$Comp
+L SW_PUSH SW2
+U 1 1 5529C4A4
+P 5950 3000
+F 0 "SW2" H 6100 3110 50  0000 C CNN
+F 1 "MODE BUTTON" H 5950 2920 50  0000 C CNN
+F 2 "~" H 5950 3000 60  0000 C CNN
+F 3 "~" H 5950 3000 60  0000 C CNN
+F 4 "C&K Components" H 5950 3000 60  0001 C CNN "Manufacturer"
+F 5 "Pushbutton SwPushbutton Switch SPST-NO Keyswitch Through Holeitch SPST-NO Keyswitch Through Hole" H 5950 3000 60  0001 C CNN "Product description"
+F 6 "D6R40 F1 LFS" H 5950 3000 60  0001 C CNN "Product code"
+F 7 "Digikey" H 5950 3000 60  0001 C CNN "Supplier"
+F 8 "401-1975-ND" H 5950 3000 60  0001 C CNN "Supplier code"
+F 9 "No" H 5950 3000 60  0001 C CNN "Order"
+F 10 "http://www.digikey.co.uk/product-detail/en/c-k-components/D6R40-F1-LFS/401-1975-ND/1466332" H 5950 3000 60  0001 C CNN "Supplier URL"
+	1    5950 3000
+	0    -1   -1   0
+$EndComp
 $EndSCHEMATC

Commit message: misc. changes
Parts:
- D1: renamed from D?; Product description Red, Green, Blue (RGB) LED Indication - Discrete 2.1V Red, 3.8V Green, 2.7V Blue 4-DIP (0.200\", 5.08mm) -> Red, Green, Blue (RGB) LED Indication - Discrete 2.1V Red, 3.8V Green, 2.7V Blue 4-DIP (0.200\" 5.08mm)
- SW2: Product description Pushbutton SwPushbutton Switch SPST-NO Keyswitch Through Ho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 -> Pushbutton Switch SPST-NO Keyswitch Through Hole
- gave numbers to parts that had none: 2
Changed lines of the file:
@@
 	6100 3550 5200 3550
 $Comp
-L CONTROLS_HEADER J?
+L CONTROLS_HEADER J1
 U 1 1 58046964
 P 4700 3850
-F 0 "J?" H 4700 2750 60  0000 C CNN
+F 0 "J1" H 4700 2750 60  0000 C CNN
 F 1 "CONTROLS_HEADER" H 4700 4500 60  0000 C CNN
 F 2 "" H 4500 3850 60  0000 C CNN
@@
 	5500 4550 5800 4550
 $Comp
-L LED_RABG D?
+L LED_RABG D1
 U 1 1 580C0207
 P 6100 4350
-F 0 "D?" H 6175 4700 50  0000 C CNN
+F 0 "D1" H 6175 4700 50  0000 C CNN
 F 1 "LED_RABG" H 6125 4000 50  0000 C CNN
 F 2 "" H 6050 4300 50  0000 C CNN
 F 3 "" H 6050 4300 50  0000 C CNN
 F 4 "Adafruit Industries LLC" H 6100 4350 60  0001 C CNN "Manufacturer"
-F 5 "Red, Green, Blue (RGB) LED Indication - Discrete 2.1V Red, 3.8V Green, 2.7V Blue 4-DIP (0.200\", 5.08mm)" H 6100 4350 60  0001 C CNN "Product description"
+F 5 "Red, Green, Blue (RGB) LED Indication - Discrete 2.1V Red, 3.8V Green, 2.7V Blue 4-DIP (0.200\" 5.08mm)" H 6100 4350 60  0001 C CNN "Product description"
 F 6 "314" H 6100 4350 60  0001 C CNN "Product code"
 F 7 "Digikey" H 6100 4350 60  0001 C CNN "Supplier"
@@
 $EndComp
 $Comp
-L SW_PUSH SW?
+L SW_PUSH SW1
 U 1 1 580D518A
 P 5600 3000
-F 0 "SW?" H 5750 3110 50  0000 C CNN
+F 0 "SW1" H 5750 3110 50  0000 C CNN
 F 1 "PARAM BUTTON" H 5600 2920 50  0000 C CNN
 F 2 "~" H 5600 3000 60  0000 C CNN
@@
 F 3 "~" H 5950 3000 60  0000 C CNN
 F 4 "C&K Components" H 5950 3000 60  0001 C CNN "Manufacturer"
-F 5 "Pushbutton SwPushbutton Switch SPST-NO Keyswitch Through Holeitch SPST-NO Keyswitch Through Hole" H 5950 3000 60  0001 C CNN "Product description"
+F 5 "Pushbutton Switch SPST-NO Keyswitch Through Hole" H 5950 3000 60  0001 C CNN "Product description"
 F 6 "D6R40 F1 LFS" H 5950 3000 60  0001 C CNN "Product code"
 F 7 "Digikey" H 5950 3000 60  0001 C CNN "Supplier"
