File: pcb/main-board/rgb-controller.sch (KiCad schematic (older format))
At the start: 23 parts, among them IC1 ATMEGA328-P, J1 LCD_HEADER, J2 CONTROL_HEADER, J3 UART_HEADER, J4 LED_HEADER, J5 PWR_IN, Q1 STP35NF10, Q2 STP35NF10, Q3 STP35NF10, SW1 SW_PUSH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

Commit message: working on finding components for parts
Parts:
- removed C4, C6, C7: 100nF, ~, symbol C-rgb
- removed C5: 22pF, ~, symbol C-RESCUE-rgb-controller
- removed J2: CONTROL_HEADER, symbol CONTROL_HEADER
- removed J5: PWR_IN, ~, symbol PWR_IN
- removed Q1, Q2, Q3: STP35NF10, symbol STP35NF10
- removed RV1: 10k, ~, symbol POT-rgb
- added C? (x3): 100nF, ~, symbol C-rgb
- added C?: 22pF, ~, symbol C-RESCUE-rgb-controller
- added F1: FUSE, symbol FUSE
- added J1: PWR_IN, symbol PWR_IN
- added J4: CONTROL_HEADER, symbol CONTROL_HEADER
- added Q4: BS170, symbol BS170
- added Q? (x3): IRL510PBF, symbol IRL510PBF
- added R2: 152R, symbol R-rgb
- added R3, R4: 85R, symbol R-rgb
- added R5: 20R, symbol R-rgb
- added RV? (x2): 20R, ~, symbol POT-rgb
- added RV?: 10k, ~, symbol POT-rgb
- C1: renamed from C2; Manufacturer Vishay -> Kemet; Order (none) -> No; Product code 489D106X0016C1VE3 -> T350E106M025AT; Product description Tantalum Capacitor, Resin Coated, 489D Series, 10 µF, ± 20%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 -> 10µF Conformal Coated Tantalum Capacitors 25V Radial 2.5 Oh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; Supplier Farnell -> Digikey; Supplier URL (none) -> http://www.digikey.co.uk/product-detail/en/kemet/T350E106M0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; Supplier code 1753975 -> 399-9907-ND
- C2: renamed from C3; Manufacturer Multicomp -> Kemet; Order (none) -> No; Product code MC0805Y104M500A2.54MM -> C315C104M5U5TA; Product description Multilayer Ceramic Capacitor, MC Series, 0.1 µF, ± 20%, Y5V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 -> 0.10µF 50V Ceramic Capacitor Z5U Radial 0.150\" L x 0.100\"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; Supplier Farnell -> Digikey; Supplier URL (none) -> http://www.digikey.co.uk/product-detail/en/kemet/C315C104M5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; Supplier code 2112751 -> 399-4151-ND
- C6: renamed from C1; Manufacturer (none) -> Kemet; Order (none) -> No; Product code (none) -> C315C220J5G5TA; Product description (none) -> 22pF 50V Ceramic Capacitor C0G, NP0 Radial 0.150\" L x 0.10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; Supplier Have -> Digikey; Supplier URL (none) -> http://www.digikey.co.uk/product-detail/en/kemet/C315C220J5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; Supplier code (none) -> 399-9721-ND
- IC1: Manufacturer Atmel -> Arduino; Order (none) -> No; Product code AT-MEGA328-P -> A000048; Supplier Have -> Digikey; Supplier URL (none) -> http://www.digikey.co.uk/product-search/en/integrated-circu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; Supplier code (none) -> 1050-1019-ND
- J2: renamed from J4; value LED_HEADER -> LED_CONNECTOR; Manufacturer (none) -> CUI Inc.; Notes (none) -> Rated to 2A per conductor at 12V DC; Order (none) -> No; Product code (none) -> MD-60S; Product description (none) -> 6 Position Circular Connector Receptacle, Female Sockets So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; Supplier (none) -> Digikey; Supplier URL (none) -> http://www.digikey.co.uk/product-detail/en/cui-inc/MD-60S/C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; Supplier code (none) -> CP-2460-ND
- R1: Manufacturer (none) -> Stackpole Electronics Inc.; Order (none) -> No; Product code (none) -> CF18JT10K0; Product description (none) -> RES 10K OHM 1/8W 5% CF AXIAL; Supplier (none) -> Digikey; Supplier URL (none) -> http://www.digikey.co.uk/product-detail/en/stackpole-electr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; Supplier code (none) -> CF18JT10K0CT-ND
- RV1: renamed from RV2; Manufacturer (none) -> Bourns Inc.; Order (none) -> No; Product code (none) -> 3362P-1-103LF; Product description (none) -> 10k Ohm 0.5W, 1/2W PC Pins Through Hole Trimmer Potentiomet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; Supplier (none) -> Digikey; Supplier URL (none) -> http://www.digikey.co.uk/product-detail/en/bourns-inc/3362P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; Supplier code (none) -> 3362P-103LF-ND
- SW1: renamed from SW2; Manufacturer (none) -> C&K Components; Order (none) -> No; Product code (none) -> E101J1AQE2; Product description (none) -> Rocker Switch SPDT 7.5A (AC/DC) 125V Through Hole, Right An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; Supplier (none) -> Digikey; Supplier URL (none) -> http://www.digikey.co.uk/product-detail/en/c-k-components/E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; Supplier code (none) -> CKN2070-ND
- U1: Manufacturer (none) -> ON Semiconductor; Order (none) -> No; Product code (none) -> NCP7805TG; Product description (none) -> Linear Voltage Regulator IC Positive Fixed 1 Output 5V 1A T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; Supplier (none) -> Digikey; Supplier URL (none) -> http://www.digikey.co.uk/product-detail/en/on-semiconductor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; Supplier code (none) -> NCP7805TGOS-ND
- renumbered J1 to J5, SW1 to SW2
Connections:
- net labels added: LIGHT
- wire segments 115 -> 159
- no-connect marks 3 -> 2
Other:
- moved on the sheet: C1, C2, C6, IC1, J2, J3, J5, R1, RV1, SW2, U1, X1

Commit message: finished choosing components for main board
Parts:
- removed Q4: BS170, symbol BS170
- removed RV?: 20R, ~, symbol POT-rgb
- removed SW2: SW_PUSH, ~, symbol SW_PUSH
- added Q4: TP0606, symbol TP0606
- added RV2: 50R, ~, symbol POT-rgb
- J3: Manufacturer (none) -> Phoenix Contact; Order (none) -> No; Product code (none) -> 1945122; Product description (none) -> 5 Position Terminal Block Header, Male Pins, Unshrouded 0.1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; Supplier (none) -> Digikey; Supplier URL (none) -> http://www.digikey.co.uk/product-detail/en/phoenix-contact/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; Supplier code (none) -> 277-1752-ND
- J4: Manufacturer (none) -> On Shore Technology Inc.; Order (none) -> No; Product code (none) -> 302-S101; Product description (none) -> 10 Positions Header, Shrouded Connector 0.100\" (2.54mm) Th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; Supplier (none) -> Digikey; Supplier URL (none) -> http://www.digikey.co.uk/product-detail/en/on-shore-technol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; Supplier code (none) -> ED1543-ND
- J5: Manufacturer (none) -> On Shore Technology Inc.; Order (none) -> No; Product code (none) -> 302-S141; Product description (none) -> 14 Positions Header, Shrouded Connector 0.100\" (2.54mm) Th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; Supplier (none) -> Digikey; Supplier URL (none) -> http://www.digikey.co.uk/product-detail/en/on-shore-technol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; Supplier code (none) -> ED10522-ND
- R2: value 152R -> 135R; Manufacturer (none) -> Stackpole Electronics Inc.; Product code (none) -> RNF18JBD130R; Product description (none) -> METAL FILM 0.125W 5% 130 OHM; Supplier (none) -> Digikey; Supplier URL (none) -> http://www.digikey.co.uk/product-detail/en/stackpole-electr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; Supplier code (none) -> 1263-RNF18JBD130R-CHP; Tolerance 1% -> 5%
- R3, R4: value 85R -> 20R; Manufacturer (none) -> Stackpole Electronics Inc.; Product code (none) -> RNF18JBD22R0; Product description (none) -> METAL FILM 0.125W 5% 22 OHM; Supplier (none) -> Digikey; Supplier URL (none) -> http://www.digikey.co.uk/product-detail/en/stackpole-electr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; Supplier code (none) -> 1263-RNF18JBD22R0-CHP
- RV3: renamed from RV?; value 20R -> 50R; Product code 3362P-1-200LF -> 3362P-1-500LF; Product description 20 Ohm 0.5W, 1/2W PC Pins Through Hole Trimmer Potentiomete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 -> 50 Ohm 0.5W, 1/2W PC Pins Through Hole Trimmer Potentiomete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; Supplier URL http://www.digikey.co.uk/product-detail/en/bourns-inc/3362P-1-200LF/3362P-1-200LF-ND/2536615 -> http://www.digikey.co.uk/product-detail/en/bourns-inc/3362P-1-500LF/3362P-1-500LF-ND/2536639; Supplier code 3362P-1-200LF-ND -> 3362P-1-500LF-ND
- X1: Manufacturer (none) -> TXC CORPORATION; Order (none) -> No; Product code (none) -> 9B-16.000MEEJ-B; Product description (none) -> 16MHz ±10ppm Crystal 18pF 30 Ohm -20°C ~ 70°C Through Hole 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; Supplier (none) -> Digikey; Supplier URL (none) -> http://www.digikey.co.uk/product-detail/en/txc-corporation/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; Supplier code (none) -> 887-1244-ND
- gave numbers to parts that had none: 8
Connections:
- net +5V: now also Q4.3 (D); no longer R5.2
- net GND: now also J5.12 (K)
- net G_GREEN: now also RV2.1, RV2.2
- net LIGHT: now also Q4.2 (G)
- net at J5.11 (A): now also R5.2; no longer R5.1
- net at J4.9 (LED_5V): now also R5.1, Q4.1 (S); no longer J5.12 (K)
- net at R3.1: now also RV2.3
Other:
- moved on the sheet: R5

Commit message: misc. changes
Parts:
- removed R4: 20R, symbol R-rgb
- added R?: 20R, symbol R-rgb
- R2: Product code RNF18JBD130R -> CF18JT130RCT-ND; Supplier URL http://www.digikey.co.uk/product-detail/en/stackpole-electronics-inc/RNF18JBD130R/1263-RNF18JBD130R-CHP/5227247 -> http://www.digikey.co.uk/product-detail/en/stackpole-electronics-inc/CF18JT130R/CF18JT130RCT-ND/2022721; Supplier code 1263-RNF18JBD130R-CHP -> CF18JT130R
- R3: Product code RNF18JBD22R0 -> CF18JT22R0; Supplier URL http://www.digikey.co.uk/product-detail/en/stackpole-electronics-inc/RNF18JBD22R0/1263-RNF18JBD22R0-CHP/5227254 -> http://www.digikey.co.uk/product-detail/en/stackpole-electronics-inc/CF18JT22R0/CF18JT22R0CT-ND/2022702; Supplier code 1263-RNF18JBD22R0-CHP -> (none)
Connections:
- net G_BLUE: no longer RV3.1, RV3.2
- net G_GREEN: no longer RV2.1, RV2.2
- net G_RED: no longer R2.1
- net LED_R: now reaches J2.1 (RED), Q1.2 (D)
- net LED_R: now also R2.1
- net LED_G: now reaches J2.2 (GREEN), Q2.2 (D)
- net LED_G: now also RV2.1, RV2.2
- net LED_B: now reaches J2.3 (BLUE), Q3.2 (D)
- net LED_B: now also RV3.1, RV3.2
- net at RV3.3: now also R?.1
- net at J4.8 (LED_B): now also R?.2
Other:
- moved on the sheet: J2
